Commit message: Lowered camera for visualization of ball

File: turtlebot3/turtlebot3_description/urdf/turtlebot3_waffle.urdf.xacro (robot description, xacro)
@@ -168,5 +168,5 @@
   </link>
   <joint name="camera_joint" type="fixed">
-    <origin xyz="0.064 -0.065 0.094" rpy="0 0 0"/>
+    <origin xyz="0.064 -0.065 0.094" rpy="0 0.2 0"/>
     <parent link="base_link"/>
     <child link="camera_link"/>
